Commit message: SysID related fixes

File: toddlerbot/descriptions/sysID_XC430/sysID_XC430.urdf (robot description, URDF)
Before this commit: robot sysID_XC430, 2 links, 1 joints
Links:
- removed link arm_430
- removed link xc430
- added link joint_0_body, mass 0.001
- added link mount_xc430, mass 0.08645; collision mesh filename=assets/merged/mount_xc430_collision.stl scale=1.0 1.0 1.0; visual mesh filename=assets/merged/mount_xc430_visual.stl scale=1.0 1.0 1.0
- added link world, mass 0.0; collision mesh filename=assets/merged/arm_430_collision.stl scale=1.0 1.0 1.0; visual mesh filename=assets/merged/arm_430_visual.stl scale=1.0 1.0 1.0
Joints:
- added joint joint_0_offset: type fixed, parent joint_0_body, child mount_xc430, origin xyz=0.0 0.0 0.0 rpy=0.0 0.0 0.0
- joint joint_0: axis 0 0 1 -> 0.0 0.0 1.0; child arm_430 -> joint_0_body; limit lower=-1.570796326794896558 upper=1.570796326794896558 effort=1 velocity=20 -> lower=-1.5707963267948966 upper=1.5707963267948966 effort=100 velocity=100; origin xyz=0.054999999999999681088 0.032699857927858962114 0.0055693959459660142761 rpy=1.57079632679489678 -5.5511151231258061214e-17 -1.5707963267948972241 -> xyz=-0.0210322 0.0551293 0.185732 rpy=3.14159 -1.5708 0.0; parent xc430 -> world
