Commit message: sysID_XC430_extended: refresh assemblies, URDFs, and motor-test rig assets
In-flight work on the extended-load sysID rig: regenerated assemblies
(arm_430 + base meshes), updated URDF/MJCF outputs, refreshed robot.yml
and config_dynamics.json, edits to assemble_xml.py and run_sysID.py for
the extended-load workflow, plus sim glue (motor_control.py, mujoco_sim.py).

This is the transitional XC430-extended rig methodology that will be
adapted to XL430 for Cobalt's actual sysID work; preserving it as the
methodology reference.

Co-Authored-By: Claude Opus 4.7 (1M context) <noreply@anthropic.com>

File: toddlerbot/descriptions/sysID_XC430_extended/sysID_XC430_extended.urdf (robot description, URDF)
Before this commit: robot sysID_XC430_extended, 5 links, 4 joints
Links:
- removed link load_large
- removed link xc430
- added link base, mass 0.1339; collision mesh filename=assets/merged/base_collision.stl scale=1.0 1.0 1.0; visual mesh filename=assets/merged/base_visual.stl scale=1.0 1.0 1.0
- link arm_430: mass 0.0154 -> 0.3549
- link world: geometry 
Joints:
- removed joint arm_4302load_large_fixed
- removed joint world2xc430_fixed
- added joint world2base_fixed: type fixed, parent world, child base, origin xyz=0.0 0.0 0.0 rpy=0.0 0.0 0.0
- joint joint_0: limit lower=-1.5707963267948948 upper=1.5707963267948983 effort=100 velocity=100 -> lower=0.0 upper=3.14159265358979 effort=100 velocity=100; origin xyz=-0.013 0.004 -0.01425 rpy=1.5708 0.0 -1.5708 -> xyz=0.0215522 -0.045682 0.372238 rpy=-3.14159 -1.5708 0.0; parent xc430 -> base
